File: Schematics/EthernetBoard_panel.brd (EAGLE design)
At the start: 160 x 60 mm, 16 parts

Commit message: restoring
Parts:
- removed U$2, U$3, U$8, U$9: XH-2, myparts:XH-2
- removed U$4: JT8P-3.2T-B10K-1-16Y, myparts:JT8P-3.2T-B10K-1-16Y
- added C5, C6: 1u, rcl:C025-025X050
- added CONTRAST: (no value), con-lstb:MA03-1
- added R6: 4.7k, rcl:0204/7
- added SW1, SW2, SW3, SW4, SW5, SW6: XH-2, myparts:XH-2
- R1: value 10k -> 4.7k; device rcl:RTRIM3339P -> rcl:0204/7
- moved R1 102.4 mm to (36.6, 43.6), turned to 180 degrees
- moved C3 98.3 mm to (13.2, 47.0), turned to 0 degrees
- moved R4 69.6 mm to (36.4, 37.5), turned to 180 degrees
- moved R3 64.6 mm to (15.7, 43.5), turned to 180 degrees
- moved C2 63.2 mm to (23.9, 47.0), turned to 0 degrees
- moved C1 42.8 mm to (34.4, 47.0), turned to 0 degrees
- moved R2 41.1 mm to (25.9, 43.5), turned to 180 degrees
- moved JP1 40.7 mm to (45.1, 32.6), flipped to the top
- moved C4 35.4 mm to (34.6, 40.4), turned to 0 degrees
- moved R5 30.8 mm to (26.0, 37.4), turned to 180 degrees
- moved U$1 4.57 mm to (8.88, 6.76), flipped to the bottom
Connections:
- new net N$2: C5.1, R5.2
- new net N$7: C6.1, R6.2
- net +5V: no longer U$4.'1, U$4.1
- net GND: now also C5.2, C6.2, CONTRAST.1, SW1.P$1, SW2.P$1, SW3.P$1, SW4.P$1, SW5.P$1, SW6.P$1; no longer R1.1, U$2.P$1, U$3.P$1, U$4.'3, U$4.3, U$8.P$1, U$9.P$1
- net LCD_SW1: now also R1.1, SW1.P$2; no longer R5.1, U$8.P$2
- net LCD_SW2: now also SW2.P$2; no longer U$9.P$2
- net LCD_SW3: now also SW3.P$2; no longer U$2.P$2
- net LCD_SW4: now also SW4.P$2; no longer U$3.P$2
- net LCD_SW5: now also R5.1, SW5.P$2; no longer U$4.2
- net LCD_SW6: now also R6.1, SW6.P$2; no longer U$4.'2
- net LCD_VO: now also CONTRAST.2; no longer R1.2
- net N$1: now also CONTRAST.3; no longer R1.3
- net N$3: now also C2.1; no longer C1.1
- net N$4: now also C3.1; no longer C2.1
- net N$5: now also C4.1; no longer C3.1
- net N$6: now also C1.1, R1.2; no longer C4.1, R5.2
Routing:
- net +5V: track 164.7 -> 37.7 mm, vias 2 -> 0
- net N$1: track 146.7 -> 44.4 mm
- net LCD_VO: track 122.3 -> 23.4 mm
- net LCD_SW4: track 111.7 -> 40.8 mm, vias 1 -> 0
- net LCD_SW6: track 0.00 -> 61.2 mm
- net LCD_SW5: track 0.00 -> 53.3 mm
- net LCD_DB7: track 0.00 -> 41.7 mm
- net LCD_DB6: track 0.00 -> 41.4 mm
- net LCD_SW3: track 89.5 -> 60.4 mm, vias 0 -> 2
- net LCD_DB3: track 13.9 -> 41.4 mm
- net LCD_DB2: track 13.9 -> 41.3 mm
- net LCD_DB5: track 13.9 -> 41.3 mm
- net LCD_DB0: track 13.9 -> 41.2 mm
- net LCD_DB4: track 13.9 -> 41.2 mm
- net LCD_DB1: track 13.9 -> 41.1 mm
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Other:
- board size 160 x 60 mm -> 50 x 50 mm
- board text added: "D48245"
