File: Schematics/EthernetBridge.sch (EAGLE design)
At the start: 55 parts, among them IC1 MEGA64-A, Q1 16.000M

Commit message: restoring
Parts:
- C5, C6, C7: value 470u -> 1000u
Changed lines of the file:
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@@
 <part name="GND23" library="SparkFun" deviceset="GND" device=""/>
 <part name="GND24" library="SparkFun" deviceset="GND" device=""/>
-<part name="C5" library="rcl" deviceset="CPOL-EU" device="E5-10.5" value="470u"/>
-<part name="C6" library="rcl" deviceset="CPOL-EU" device="E5-10.5" value="470u"/>
-<part name="C7" library="rcl" deviceset="CPOL-EU" device="E5-10.5" value="470u"/>
+<part name="C5" library="rcl" deviceset="CPOL-EU" device="E5-10.5" value="1000u"/>
+<part name="C6" library="rcl" deviceset="CPOL-EU" device="E5-10.5" value="1000u"/>
+<part name="C7" library="rcl" deviceset="CPOL-EU" device="E5-10.5" value="1000u"/>
 <part name="GND25" library="SparkFun" deviceset="GND" device=""/>
 <part name="GND26" library="SparkFun" deviceset="GND" device=""/>
