File: Schematics/PointController.sch (EAGLE design)
At the start: 114 parts, among them IC1 MEGA48/88/168-AU

Commit message: create route test; board edit
Parts:
- added C38, C4: (no value), rcl:C-EUC1608
- added R43, R44, R45, R46, R47, R48, R49: 100k, rcl:R-EU_R0603
- added U$30, U$31, U$32, U$33, U$34, U$35, U$36, U$37, U$38, U$39: POLYSWITCH_20204/5, myparts:POLYSWITCH_20204/5
- IC1: value MEGA48/88/168-AU -> MEGA164P/324P/644P-AU; device avr-7:MEGA48/88/168-AU -> avr-7:MEGA164P/324P/644P-AU
- JP1: value AVR-ISP-10 -> AVR-JTAG-10; device avr-7:AVR-ISP-10 -> avr-7:AVR-JTAG-10
- R1, R13, R18, R23, R28, R3, R33, R38, R8: device rcl:R-US_M3216 -> rcl:R-EU_R0603
- R10, R11, R15, R16, R20, R21, R25, R26, R30, R31, R35, R36, R40, R41, R5, R6: value 10k -> 100k; device rcl:R-US_M3216 -> rcl:R-EU_R0603
- R2: value (none) -> 100k; device rcl:R-EU_0922/22 -> rcl:R-EU_R0603
Connections:
- removed net PT_PWR: C10.+, C14.+, C18.+, C22.+, C26.+, C30.+, C34.+, C6.+, R13.2, R18.2, R2.1, R23.2, R28.2, R3.2, R33.2, R38.2, R8.2, U$1.VS, U$11.VS, U$14.VS, U$17.VS, U$20.VS, U$23.VS, U$26.VS, U$8.VS
- new net N$43: U$2.1_12V, U$2.2_12V, U$2.4_12V, U$31.1
- new net N$44: C37.+, U$2.6_5V, U$32.1
- new net N$45: C6.+, R3.2, U$1.VS, U$30.1
- new net N$46: C14.+, R13.2, U$11.VS, U$34.1
- new net N$47: C22.+, R23.2, U$17.VS, U$36.1
- new net N$48: C30.+, R33.2, U$23.VS, U$38.1
- new net N$49: C34.+, R38.2, U$26.VS, U$39.1
- new net N$50: C26.+, R28.2, U$20.VS, U$37.1
- new net N$51: C18.+, R18.2, U$14.VS, U$35.1
- new net N$52: C10.+, R8.2, U$33.1, U$8.VS
- new net TCK: IC1.(TCK/PCINT18)PC2, JP1.1
- new net TDI: IC1.(TDI/PCINT21)PC5, JP1.9
- new net TDO: IC1.(TDO/PCINT20)PC4, JP1.3
- new net TMS: IC1.(TMS/PCINT19)PC3, JP1.5
- net !RESET: now also IC1.!RESET, JP1.6; no longer IC1.PC6(/RESET/PCINT14), JP1.5
- net !SS: now also IC1.(OC0B/!SS!/PCINT12)PB4; no longer IC1.PB2(SS/OC1B/PCINT2)
- net +12V: now also U$30.2, U$31.2, U$33.2, U$34.2, U$35.2, U$36.2, U$37.2, U$38.2, U$39.2; no longer R2.2, U$2.1_12V, U$2.2_12V, U$2.4_12V
- net 5V: now also C38.1, C4.1, IC1.VCC@3, JP1.4, JP1.7, U$32.2; no longer C37.+, JP1.2, U$2.6_5V
- net GND: now also C38.2, C4.2, IC1.GND@3, IC1.GND@4, JP1.2, R2.2, R43.2, R44.2, R45.2, R46.2, R47.2, R48.2, R49.2; no longer IC1.AGND, JP1.3, JP1.4, JP1.6, JP1.8
- net MISO: now also IC1.(MISO/PCINT14)PB6; no longer IC1.PB4(MISO/PCINT4), JP1.9
- net MOSI: now also IC1.(MOSI/PCINT13)PB5; no longer IC1.PB3(MOSI/OC2A/PCINT3), JP1.1
- net N$13: now also R44.1
- net N$18: now also R45.1
- net N$2: now also R43.1
- net N$23: now also R46.1
- net N$28: now also R47.1
- net N$3: now also IC1.XTAL1; no longer IC1.PB7(XTAL2/TOSC2/PCINT7)
- net N$33: now also R48.1
- net N$38: now also R49.1
- net N$4: now also IC1.XTAL2; no longer IC1.PB6(XTAL1/TOSC1/PCINT6)
- net N$6: now also R2.1
- net OUT_A_0: now also IC1.(ADC0/PCINT0)PA0; no longer IC1.PC0(ADC0/PCINT8)
- net OUT_A_1: now also IC1.(ADC1/PCINT1)PA1; no longer IC1.PC1(ADC1/PCINT9)
- net OUT_B_0: now also IC1.(ADC2/PCINT2)PA2; no longer IC1.PC2(ADC2/PCINT10)
- net OUT_B_1: now also IC1.(ADC3/PCINT3)PA3; no longer IC1.PC3(ADC3/PCINT11)
- net OUT_C_0: now also IC1.(ADC4/PCINT4)PA4; no longer IC1.PC4(ADC4/SDA/PCINT12)
- net OUT_C_1: now also IC1.(ADC5/PCINT5)PA5; no longer IC1.PC5(ADC5/SCL/PCINT13)
- net OUT_D_0: now also IC1.(ADC6/PCINT6)PA6; no longer IC1.PD0(RXD/PCINT16)
- net OUT_D_1: now also IC1.(ADC7/PCINT7)PA7; no longer IC1.PD1(TXD/PCINT17)
- net OUT_E_0: now also IC1.(RXD0/PCINT24)PD0; no longer IC1.PD2(INT0/PCINT18)
- net OUT_E_1: now also IC1.(TXD0/PCINT25)PD1; no longer IC1.PD3(INT1/OC2B/PCINT19)
- net OUT_F_0: now also IC1.(RXD1/INT0/PCINT26)PD2; no longer IC1.PD4(T0/XCK/PCINT20)
- net OUT_F_1: now also IC1.(TXD1/INT1/PCINT27)PD3; no longer IC1.PD5(T1/OC0B/PCINT21)
- net OUT_G_0: now also IC1.(XCK1/OC1B/PCINT28)PD4; no longer IC1.PD6(AIN0/OC0A/PCINT22)
- net OUT_G_1: now also IC1.(OC1A/PCINT29)PD5; no longer IC1.PD7(AIN1/PCINT23)
- net OUT_H_0: now also IC1.(OC2B/ICP/PCINT30)PD6; no longer IC1.PB0(ICP1/CLKO/PCINT0)
- net OUT_H_1: now also IC1.(OC2A/PCINT31)PD7; no longer IC1.PB1(OC1A/PCINT1)
- net SCK: now also IC1.(SCK/PCINT15)PB7; no longer IC1.PB5(SCK/PCINT5), JP1.7
Other:
- moved on the sheet: JP1, R2

Commit message: restoring
Parts:
- removed C32, C36: (no value), capacitor-wima:C5/3
- removed C33: 10u, resistor:CPOL-EUE1.8-4
- removed C34, C37: 47u, resistor:CPOL-EUE1.8-4
- removed C38: (no value), rcl:C-EUC1608
- removed U$31, U$32: POLYSWITCH_20204/5, myparts:POLYSWITCH_20204/5
- removed U$8: TA7291, TA7291P:TA7291
- added C100, C101, C102, C104, C105, C106, C107: 0.1u, rcl:C-EUC1608
- added F7: POLYSWITCH_20204/5, myparts:POLYSWITCH_20204/5
- added IC6: MEGA164P/324P/644P-AU, avr-7:MEGA164P/324P/644P-AU
- C1, C2: value (none) -> 47u; device rcl:C-EUC1608 -> capacitor-wima:C5/3
- C10, C14, C18, C30, C6: value 47u -> 0.1u; device resistor:CPOL-EUE1.8-4 -> rcl:C-EUC1608
- C12, C28, C8: value (none) -> 47u
- C13, C29, C9: value 10u -> (none); device resistor:CPOL-EUE1.8-4 -> rcl:CPOL-EUE2.5-5
- C16, C24: device capacitor-wima:C5/3 -> rcl:CPOL-EUE2.5-5
- C17, C25, C5: value 10u -> 0.1u; device resistor:CPOL-EUE1.8-4 -> rcl:C-EUC1608
- C19, C7: value 0.1u -> 47u; device rcl:C-EUC1608 -> capacitor-wima:C5/3
- C20: value (none) -> 22p; device capacitor-wima:C5/3 -> rcl:C-EUC1608
- C21: value 10u -> 22p; device resistor:CPOL-EUE1.8-4 -> rcl:C-EUC1608
- C22: device resistor:CPOL-EUE1.8-4 -> rcl:CPOL-EUE2.5-5
- C23: value 0.1u -> 47u; device rcl:C-EUC1608 -> rcl:CPOL-EUE2.5-5
- C26: device resistor:CPOL-EUE1.8-4 -> capacitor-wima:C5/3
- C27: value 0.1u -> (none); device rcl:C-EUC1608 -> rcl:CPOL-EUE2.5-5
- C3, C4: device rcl:C-EUC1608 -> rcl:CPOL-EUE2.5-5
- IC1: value MEGA164P/324P/644P-AU -> TA7291; device avr-7:MEGA164P/324P/644P-AU -> TA7291P:TA7291
- LED1, LED11, LED13, LED15, LED3, LED5, LED7, LED9: value (none) -> G
- LED10, LED12, LED14, LED16, LED2, LED4, LED6, LED8: value (none) -> O
- Q1: value (none) -> 20.000M
- R1: value (none) -> 10k; device rcl:R-EU_R0603 -> resistor:R-EU_0204/7
- R10, R21, R36, R46, R47: value 100k -> 1k; device rcl:R-EU_R0603 -> resistor:R-EU_R0603
- R12, R17, R24, R37, R42: value (none) -> 100k; device resistor:R-EU_0204/7 -> rcl:R-EU_R0603
- R13, R38: device rcl:R-EU_R0603 -> resistor:R-EU_0204/7
- R14, R32, R39: value (none) -> 10k
- R16, R31, R41, R43: value 100k -> 10k
- R18, R23, R28, R3, R33, R8: value 10k -> 100k
- R19, R27, R34, R4, R7: value (none) -> 10k; device resistor:R-EU_0204/7 -> rcl:R-EU_R0603
- R2, R25: value 100k -> 10k; device rcl:R-EU_R0603 -> resistor:R-EU_0204/7
- R22, R29, R9: value (none) -> 1k; device resistor:R-EU_0204/7 -> resistor:R-EU_R0603
- renumbered C35 to C103, U$1 to IC4, U$10 to B, U$11 to IC2, U$13 to C, U$14 to IC3, U$16 to D, U$17 to IC9, U$19 to E, U$2 to CONN, U$20 to IC8, U$22 to F, U$23 to IC7, U$25 to G, U$26 to IC5, U$28 to H, U$30 to F3, U$33 to F1, U$34 to F2, U$35 to F4, U$36 to F8, U$37 to F9, U$38 to F6, U$39 to F5, U$7 to A
Connections:
- removed net N$43: CONN.1_12V, CONN.2_12V, CONN.4_12V, U$31.1
- net !RESET: now also IC6.!RESET, R31.2; no longer IC1.!RESET, R1.2
- net !SS: now also IC6.(OC0B/!SS!/PCINT12)PB4; no longer IC1.(OC0B/!SS!/PCINT12)PB4
- net +12V: now also C22.+, CONN.1_12V, CONN.2_12V, CONN.4_12V; no longer U$31.2
- net 5V: now also C100.2, C101.2, C102.2, C104.2, C105.2, C106.2, C107.2, C14.1, C17.1, C18.1, C23.+, F7.2, IC1.VCC, IC6.AREF, IC6.AVCC, IC6.VCC@1, IC6.VCC@2, IC6.VCC@3, R31.1; no longer C11.2, C13.+, C15.2, C17.+, C19.2, C21.+, C23.2, C25.+, C27.2, C29.+, C3.1, C31.2, C33.+, C38.1, C4.1, C5.+, C7.2, C9.+, IC1.AVCC, IC1.VCC@1, IC1.VCC@2, IC1.VCC@3, R1.1, U$32.2, U$8.VCC
- net GND: now also C10.1, C100.1, C101.1, C102.1, C104.1, C105.1, C106.1, C107.1, C14.2, C16.-, C17.2, C18.2, C20.1, C21.1, C23.-, C24.-, C25.1, C27.-, C3.-, C30.1, C4.-, C5.1, C6.1, IC1.GND, IC6.GND@1, IC6.GND@2, IC6.GND@3, IC6.GND@4, R12.1, R15.2, R17.1, R18.2, R23.1, R24.1, R26.2, R28.1, R3.2, R33.2, R37.1, R40.2, R42.1, R45.1, R48.1, R49.1, R6.2, R8.1; no longer C1.1, C10.-, C14.-, C17.-, C18.-, C19.1, C2.1, C21.-, C23.1, C25.-, C26.-, C27.1, C3.2, C30.-, C33.-, C34.-, C37.-, C38.2, C4.2, C5.-, C6.-, C7.1, IC1.GND@1, IC1.GND@2, IC1.GND@3, IC1.GND@4, R10.1, R15.1, R16.1, R2.2, R21.1, R25.1, R26.1, R31.1, R36.1, R40.1, R41.1, R43.2, R45.2, R46.2, R47.2, R48.2, R49.2, R6.1, U$8.GND
- net MISO: now also IC6.(MISO/PCINT14)PB6; no longer IC1.(MISO/PCINT14)PB6
- net MOSI: now also IC6.(MOSI/PCINT13)PB5; no longer IC1.(MOSI/PCINT13)PB5
- net N$1: now also LED5.C, LED6.A, R22.2; no longer LED1.A, LED2.C, R7.2
- net N$10: now also IC1.OUT2, R1.1, R10.1; no longer R12.1, R9.1, U$8.OUT2
- net N$11: now also C1.1, R1.2; no longer C12.1, R9.2
- net N$12: now also LED3.C, LED4.A, R10.2; no longer LED3.A, LED4.C, R12.2
- net N$13: now also R3.1, R4.1; no longer R13.1, R44.1
- net N$14: now also C2.2, LED1.A, LED2.C; no longer C16.2, LED5.C, LED6.A
- net N$15: now also R2.1, R9.1; no longer R14.1, R17.1
- net N$16: now also C2.1, R2.2; no longer C16.1, R14.2
- net N$17: now also LED1.C, LED2.A, R9.2; no longer LED5.A, LED6.C, R17.2
- net N$18: now also R15.1, R16.1; no longer R18.1, R45.1
- net N$19: now also C8.2, LED7.A, LED8.C; no longer C20.2, LED7.C, LED8.A
- net N$2: now also IC1.VREF, R6.1, R7.1; no longer R43.1, R8.1, U$8.VREF
- net N$20: now also R14.1, R21.1; no longer R19.1, R22.1
- net N$21: now also C8.1, R14.2; no longer C20.1, R19.2
- net N$22: now also LED7.C, LED8.A, R21.2; no longer LED7.A, LED8.C, R22.2
- net N$23: now also R43.1, R44.1; no longer R23.1, R46.1
- net N$24: now also C26.2, LED13.A, LED14.C; no longer C24.2, LED10.A, LED9.C
- net N$25: now also R38.1, R47.1; no longer R24.1, R27.1
- net N$26: now also C26.1, R38.2; no longer C24.1, R24.2
- net N$27: now also LED13.C, LED14.A, R47.2; no longer LED10.C, LED9.A, R27.2
- net N$28: now also R40.1, R41.1; no longer R28.1, R47.1
- net N$29: now also LED15.A, LED16.C; no longer LED11.C, LED12.A
- net N$3: now also C20.2, IC6.XTAL1; no longer C1.2, IC1.XTAL1
- net N$30: now also R39.1, R46.1; no longer R29.1, R32.1
- net N$31: now also R39.2; no longer R29.2
- net N$32: now also LED15.C, LED16.A, R46.2; no longer LED11.A, LED12.C, R32.2
- net N$33: now also R34.1; no longer R48.1
- net N$34: now also C19.2, LED11.A, LED12.C; no longer C32.2, LED13.C, LED14.A
- net N$35: now also R32.1, R36.1; no longer R34.1, R37.1
- net N$36: now also C19.1, R32.2; no longer C32.1, R34.2
- net N$37: now also LED11.C, LED12.A, R36.2; no longer LED13.A, LED14.C, R37.2
- net N$38: now also R26.1, R27.1; no longer R38.1, R49.1
- net N$39: now also C12.2, LED10.C, LED9.A; no longer C36.2, LED15.C, LED16.A
- net N$4: now also C21.2, IC6.XTAL2; no longer C2.2, IC1.XTAL2
- net N$40: now also R25.1, R29.1; no longer R39.1, R42.1
- net N$41: now also C12.1, R25.2; no longer C36.1, R39.2
- net N$42: now also LED10.A, LED9.C, R29.2; no longer LED15.A, LED16.C, R42.2
- net N$44: now also F7.1; no longer C37.+, U$32.1
- net N$45: now also C11.2, C13.+, R19.2; no longer C6.+, R3.2
- net N$46: now also C4.+, C5.2, R4.2; no longer C14.+, R13.2
- net N$47: now also C27.+, C31.2, R43.2; no longer C22.+, R23.2
- net N$48: now also C24.+, C25.2, R34.2; no longer C30.+, R33.2
- net N$49: now also C15.2, C16.+, R27.2; no longer C34.+, R38.2
- net N$5: now also C1.2, IC1.OUT1, LED3.A, LED4.C; no longer C12.2, LED3.C, LED4.A, U$8.OUT1
- net N$50: now also C29.+, C30.2, R41.2; no longer C26.+, R28.2
- net N$51: now also C10.2, C9.+, R16.2; no longer C18.+, R18.2
- net N$52: now also C3.+, C6.2, IC1.VS, R7.2; no longer C10.+, R8.2, U$8.VS
- net N$6: now also R18.1, R19.1; no longer R2.1, R3.1
- net N$7: now also C7.2, LED5.A, LED6.C; no longer C8.2, LED1.C, LED2.A
- net N$8: now also R13.1, R22.1; no longer R4.1, R7.1
- net N$9: now also C7.1, R13.2; no longer C8.1, R4.2
- net OUT_A_0: now also IC6.(ADC0/PCINT0)PA0, R20.2; no longer IC1.(ADC0/PCINT0)PA0, R5.2
- net OUT_A_1: now also IC6.(ADC1/PCINT1)PA1, R24.2; no longer IC1.(ADC1/PCINT1)PA1, R6.2
- net OUT_B_0: now also IC1.IN1, IC6.(ADC2/PCINT2)PA2, R12.2; no longer IC1.(ADC2/PCINT2)PA2, R10.2, U$8.IN1
- net OUT_B_1: now also IC1.IN2, IC6.(ADC3/PCINT3)PA3, R8.2; no longer IC1.(ADC3/PCINT3)PA3, R11.2, U$8.IN2
- net OUT_C_0: now also IC6.(ADC4/PCINT4)PA4, R5.2; no longer IC1.(ADC4/PCINT4)PA4, R15.2
- net OUT_C_1: now also IC6.(ADC5/PCINT5)PA5, R11.2; no longer IC1.(ADC5/PCINT5)PA5, R16.2
- net OUT_D_0: now also IC6.(ADC6/PCINT6)PA6, R17.2; no longer IC1.(ADC6/PCINT6)PA6, R20.2
- net OUT_D_1: now also IC6.(ADC7/PCINT7)PA7, R23.2; no longer IC1.(ADC7/PCINT7)PA7, R21.2
- net OUT_E_0: now also IC6.(RXD0/PCINT24)PD0, R45.2; no longer IC1.(RXD0/PCINT24)PD0, R25.2
- net OUT_E_1: now also IC6.(TXD0/PCINT25)PD1, R49.2; no longer IC1.(TXD0/PCINT25)PD1, R26.2
- net OUT_F_0: now also IC6.(RXD1/INT0/PCINT26)PD2, R48.2; no longer IC1.(RXD1/INT0/PCINT26)PD2, R30.2
- net OUT_F_1: now also IC6.(TXD1/INT1/PCINT27)PD3, R42.2; no longer IC1.(TXD1/INT1/PCINT27)PD3, R31.2
- net OUT_G_0: now also IC6.(XCK1/OC1B/PCINT28)PD4, R37.2; no longer IC1.(XCK1/OC1B/PCINT28)PD4, R35.2
- net OUT_G_1: now also IC6.(OC1A/PCINT29)PD5, R35.2; no longer IC1.(OC1A/PCINT29)PD5, R36.2
- net OUT_H_0: now also IC6.(OC2B/ICP/PCINT30)PD6, R30.2; no longer IC1.(OC2B/ICP/PCINT30)PD6, R40.2
- net OUT_H_1: now also IC6.(OC2A/PCINT31)PD7, R28.2; no longer IC1.(OC2A/PCINT31)PD7, R41.2
- net SCK: now also IC6.(SCK/PCINT15)PB7; no longer IC1.(SCK/PCINT15)PB7
- net TCK: now also IC6.(TCK/PCINT18)PC2; no longer IC1.(TCK/PCINT18)PC2
- net TDI: now also IC6.(TDI/PCINT21)PC5; no longer IC1.(TDI/PCINT21)PC5
- net TDO: now also IC6.(TDO/PCINT20)PC4; no longer IC1.(TDO/PCINT20)PC4
- net TMS: now also IC6.(TMS/PCINT19)PC3; no longer IC1.(TMS/PCINT19)PC3
Other:
- moved on the sheet: C1, C11, C12, C13, C15, C19, C2, C20, C22, C29, C31, C7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
