File: Schematics/Box/Box_Bottom.brd (EAGLE design)
At the start: 300 x 190 mm, 0 parts

Commit message: restore repository
Changed lines of the file:
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@@
 <wire x1="295" y1="100" x2="295" y2="180" width="0.4064" layer="20"/>
 <wire x1="295" y1="180" x2="205" y2="180" width="0.4064" layer="20"/>
-<hole x="210" y="175" drill="3"/>
-<hole x="210" y="105" drill="3"/>
-<hole x="290" y="105" drill="3"/>
-<hole x="290" y="175" drill="3"/>
+<hole x="210" y="175" drill="3.2"/>
+<hole x="210" y="105" drill="3.2"/>
+<hole x="290" y="105" drill="3.2"/>
+<hole x="290" y="175" drill="3.2"/>
 <wire x1="205" y1="90" x2="205" y2="10" width="0.4064" layer="20"/>
 <wire x1="205" y1="10" x2="295" y2="10" width="0.4064" layer="20"/>
 <wire x1="295" y1="10" x2="295" y2="90" width="0.4064" layer="20"/>
 <wire x1="295" y1="90" x2="205" y2="90" width="0.4064" layer="20"/>
-<hole x="210" y="85" drill="3"/>
-<hole x="210" y="15" drill="3"/>
-<hole x="290" y="15" drill="3"/>
-<hole x="290" y="85" drill="3"/>
+<hole x="210" y="85" drill="3.2"/>
+<hole x="210" y="15" drill="3.2"/>
+<hole x="290" y="15" drill="3.2"/>
+<hole x="290" y="85" drill="3.2"/>
 <wire x1="105" y1="180" x2="105" y2="100" width="0.4064" layer="20"/>
 <wire x1="105" y1="100" x2="195" y2="100" width="0.4064" layer="20"/>
 <wire x1="195" y1="100" x2="195" y2="180" width="0.4064" layer="20"/>
 <wire x1="195" y1="180" x2="105" y2="180" width="0.4064" layer="20"/>
-<hole x="110" y="175" drill="3"/>
-<hole x="110" y="105" drill="3"/>
-<hole x="190" y="105" drill="3"/>
-<hole x="190" y="175" drill="3"/>
+<hole x="110" y="175" drill="3.2"/>
+<hole x="110" y="105" drill="3.2"/>
+<hole x="190" y="105" drill="3.2"/>
+<hole x="190" y="175" drill="3.2"/>
 <wire x1="105" y1="90" x2="105" y2="10" width="0.4064" layer="20"/>
 <wire x1="105" y1="10" x2="195" y2="10" width="0.4064" layer="20"/>
 <wire x1="195" y1="10" x2="195" y2="90" width="0.4064" layer="20"/>
 <wire x1="195" y1="90" x2="105" y2="90" width="0.4064" layer="20"/>
-<hole x="110" y="85" drill="3"/>
-<hole x="110" y="15" drill="3"/>
-<hole x="190" y="15" drill="3"/>
-<hole x="190" y="85" drill="3"/>
+<hole x="110" y="85" drill="3.2"/>
+<hole x="110" y="15" drill="3.2"/>
+<hole x="190" y="15" drill="3.2"/>
+<hole x="190" y="85" drill="3.2"/>
 <wire x1="5" y1="180" x2="85" y2="180" width="0.4064" layer="20"/>
 <wire x1="85" y1="180" x2="85" y2="10" width="0.4064" layer="20"/>
 <wire x1="85" y1="10" x2="5" y2="10" width="0.4064" layer="20"/>
 <wire x1="5" y1="10" x2="5" y2="180" width="0.4064" layer="20"/>
-<hole x="10" y="175" drill="3"/>
-<hole x="80" y="175" drill="3"/>
-<hole x="10" y="15" drill="3"/>
-<hole x="80" y="15" drill="3"/>
+<hole x="10" y="175" drill="3.2"/>
+<hole x="80" y="175" drill="3.2"/>
+<hole x="10" y="15" drill="3.2"/>
+<hole x="80" y="15" drill="3.2"/>
 </plain>
 <attributes>
