File: Schematics/EthControlling/SensorController_revB.brd (EAGLE design)
At the start: 90 x 80 mm, 40 parts, among them IC2 MEGA164P/324P/644P-AU, IC4 4066D, Q1 20.000M, T1 2SC1815, T3 2SC1815, T5 2SC1815, T6 2SC1815

Commit message: ditto
Parts:
- removed A_OUT1: SERIAL_SENSORXH, myparts:XH-5
- removed C9: (no value), rcl:E2,5-5
- removed F4: POLYSWITCH, myparts:0207/2V
- removed L2: (no value), rcl:0207/10
- removed R5: 1k, rcl:R0603
- removed R6: (no value), rcl:0207/7
- removed T2: (no value), zetex:SO8
- removed T3, T5, T6: 2SC1815, myparts:TO92-ECB
- removed U$1: TLP621-2, myparts:SOCKET-08
- added B_OUT: SERIAL_SENSORXH, myparts:XH-5
- added T4: (no value), zetex:SOT-23
- R1, R4: value 1k -> 100k
- R10, R3, R9: value 1k -> 10k
- R11, R12, R7, R8: value 330 -> 1k
- R2: value (none) -> 10k; device rcl:0207/7 -> rcl:R0603
- T1: value 2SC1815 -> (none); device myparts:TO92-ECB -> zetex:SOT-23
- moved R12 79.5 mm to (58.9, 30.9)
- moved R11 75.5 mm to (59.3, 28.9)
- moved R8 55.6 mm to (30.1, 34.5)
- moved R7 53.2 mm to (30.1, 36.6)
- moved F1 26.6 mm to (28.9, 67.5)
- moved R4 22.0 mm to (41.9, 67.9), turned to 270 degrees
- moved C10 21.8 mm to (25.6, 50.0), turned to 0 degrees
- moved IC4 17.2 mm to (25.2, 55.3), turned to 270 degrees
- moved R2 13.6 mm to (35.4, 67.9), turned to 270 degrees
- moved R3 12.6 mm to (32.5, 67.9), turned to 270 degrees
- moved R9 12.1 mm to (17.0, 68.0), turned to 270 degrees
- moved R10 9.46 mm to (14.3, 67.9), turned to 270 degrees
- moved R1 9.09 mm to (23.2, 67.9), turned to 270 degrees
- moved R39 8.61 mm to (29.9, 39.0)
- moved T1 7.02 mm to (38.6, 67.9)
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Connections:
- removed net +12V: L2.2, R2.2, R6.2, U$1.6, U$1.8
- removed net N$11: R5.2, U$1.3
- removed net N$12: T5.B, T5.C, T6.B, U$1.5
- removed net N$13: R6.1, T2.4, T6.C
- removed net N$14: A_OUT1.4, IC4.10, R3.1
- removed net N$15: A_OUT1.3, IC4.9, R4.1
- removed net N$16: C9.+, F1.2, L2.1
- removed net N$19: A_OUT1.2, F4.1, T2.6
- removed net N$8: R2.1, T2.2, T3.C
- net +5V: now also F1.2, R2.2; no longer F4.2, R4.2
- net A_LED: now also IC2.35, R1.2, T4.3; no longer IC2.36, R1.1
- net A_SET: now also IC2.34; no longer IC2.37
- net B_LED: now also IC2.36, R4.2, T1.3; no longer IC2.35, R5.1
- net B_SET: now also IC2.37; no longer IC2.34
- net GND: now also B_OUT.5, R1.1, R4.1, T1.2, T4.2; no longer A_OUT1.5, C9.-, T1.E, T3.E, T5.E, T6.E, U$1.2, U$1.4
- net N$1: now also T4.1; no longer T2.1
- net N$10: now also IC4.3; no longer IC4.2
- net N$18: no longer T2.8
- net N$3: now also B_OUT.4, IC4.9, R2.1; no longer CONN1.1, CONN1.2, CONN1.4, F1.1
- net N$5: now also B_OUT.3, IC4.10, R3.1; no longer R1.2, U$1.1
- net N$6: now also B_OUT.2, F1.1; no longer T1.B, T1.C, T3.B, U$1.7
- net N$7: now also B_OUT.1, T1.1; no longer A_OUT1.1, T2.3
- net N$9: now also IC4.2; no longer IC4.3
- net RX0: now also IC4.11, IC4.4; no longer IC4.1, IC4.8
- net TX0: now also IC4.1, IC4.8; no longer IC4.11, IC4.4

Commit message: ditto
Parts:
- added A_OUT1, A_OUT2, A_OUT3, B_OUT1, B_OUT2, B_OUT3: SERIAL_SENSORXH, myparts:XH-5
- added C4, C5, C9: 0.1u, rcl:C1608
- added F4, F5, F6, F7, F8, F9: POLYSWITCH, myparts:0207/2V
- added IC1, IC3, IC5: 4066D, 40xx:SO14
- added R13, R16, R19, R22, R25, R28: 100k, rcl:R0603
- added R14, R15, R17, R18, R20, R21, R23, R24, R26, R27, R5, R6: 10k, rcl:R0603
- added T2, T3, T5, T6, T7, T8: (no value), zetex:SOT-23
Connections:
- new net N$11: A_OUT1.3, IC1.3, R6.1
- new net N$12: A_OUT1.2, F4.1
- new net N$13: A_OUT1.1, T2.1
- new net N$14: B_OUT1.4, IC1.9, R14.1
- new net N$15: B_OUT1.3, IC1.10, R15.1
- new net N$16: B_OUT1.2, F5.1
- new net N$19: B_OUT1.1, T3.1
- new net N$24: A_OUT2.4, IC3.2, R17.1
- new net N$25: A_OUT2.3, IC3.3, R18.1
- new net N$26: A_OUT2.2, F6.1
- new net N$27: A_OUT2.1, T5.1
- new net N$28: B_OUT2.4, IC3.9, R20.1
- new net N$29: B_OUT2.3, IC3.10, R21.1
- new net N$30: B_OUT2.2, F7.1
- new net N$31: B_OUT2.1, T6.1
- new net N$32: A_OUT3.4, IC5.2, R23.1
- new net N$33: A_OUT3.3, IC5.3, R24.1
- new net N$34: A_OUT3.2, F8.1
- new net N$35: A_OUT3.1, T7.1
- new net N$36: B_OUT3.4, IC5.9, R26.1
- new net N$37: B_OUT3.3, IC5.10, R27.1
- new net N$38: B_OUT3.2, F9.1
- new net N$39: B_OUT3.1, T8.1
- new net N$8: A_OUT1.4, IC1.2, R5.1
- net +5V: now also C4.2, C5.2, C9.2, F4.2, F5.2, F6.2, F7.2, F8.2, F9.2, IC1.14, IC3.14, IC5.14, R14.2, R15.2, R17.2, R18.2, R20.2, R21.2, R23.2, R24.2, R26.2, R27.2, R5.2, R6.2
- net A_LED: now also R13.2, R19.2, R25.2, T2.3, T5.3, T7.3
- net A_SET: now also IC1.13, IC1.5, IC3.13, IC3.5, IC5.13, IC5.5
- net B_LED: now also R16.2, R22.2, R28.2, T3.3, T6.3, T8.3
- net B_SET: now also IC1.12, IC1.6, IC3.12, IC3.6, IC5.12, IC5.6
- net GND: now also A_OUT1.5, A_OUT2.5, A_OUT3.5, B_OUT1.5, B_OUT2.5, B_OUT3.5, C4.1, C5.1, C9.1, IC1.7, IC3.7, IC5.7, R13.1, R16.1, R19.1, R22.1, R25.1, R28.1, T2.2, T3.2, T5.2, T6.2, T7.2, T8.2
- net RX0: now also IC1.11, IC1.4, IC3.11, IC3.4, IC5.11, IC5.4
- net TX0: now also IC1.1, IC1.8, IC3.1, IC3.8, IC5.1, IC5.8

Commit message: ditto
Parts:
- moved C5 12.3 mm to (25.2, 19.9)
- moved R25 10.2 mm to (48.4, 13.8)
- moved R19 9.75 mm to (11.4, 13.8)
- moved R28 8.98 mm to (66.6, 13.8)
- moved R18 8.53 mm to (20.3, 13.8), turned to 270 degrees
- moved R11 7.98 mm to (51.6, 26.8), turned to 180 degrees
- moved R12 7.42 mm to (51.6, 29.7), turned to 180 degrees
- moved R23 5.70 mm to (54.9, 13.8), turned to 270 degrees
- moved R26 5.70 mm to (73.2, 13.8), turned to 270 degrees
- moved Q1 4.76 mm to (42.2, 28.1)
- moved C7 4.38 mm to (39.1, 31.6)
- moved C8 4.38 mm to (42.6, 31.6)
- moved R27 2.96 mm to (75.6, 13.8), turned to 270 degrees
- moved F9 2.57 mm to (79.2, 13.8)
- moved R24 2.19 mm to (57.7, 13.8), turned to 270 degrees
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- renumbered A_OUT1 to C_OUT, A_OUT2 to E_OUT, A_OUT3 to G_OUT, B_OUT1 to D_OUT, B_OUT2 to F_OUT, B_OUT3 to H_OUT
Connections:
- removed net TRANS_STANDBY: IC2.13
- net A_LED: no longer R13.2, R19.2, R25.2, T2.3, T5.3, T7.3
- net A_SET: now also IC2.36; no longer IC1.13, IC1.5, IC2.34, IC3.13, IC3.5, IC5.13, IC5.5
- net B_LED: now also IC2.34; no longer IC2.36, R16.2, R22.2, R28.2, T3.3, T6.3, T8.3
- net B_SET: no longer IC1.12, IC1.6, IC3.12, IC3.6, IC5.12, IC5.6
- net C_LED: now also R13.2, T2.3
- net C_SET: now also IC1.13, IC1.5
- net D_LED: now also R16.2, T3.3
- net D_SET: now also IC1.12, IC1.6
- net E_LED: now also R19.2, T5.3
- net E_SET: now also IC3.13, IC3.5
- net F_LED: now also R22.2, T6.3
- net F_SET: now also IC3.12, IC3.6
- net G_LED: now also IC2.13, R25.2, T7.3; no longer IC2.20
- net G_SET: now also IC2.16, IC5.13, IC5.5; no longer IC2.19
- net H_LED: now also IC2.14, R28.2, T8.3; no longer IC2.25
- net H_SET: now also IC2.15, IC5.12, IC5.6; no longer IC2.26
- net RX0: no longer IC3.11, IC3.4, IC5.11, IC5.4
- net RX1: now also IC3.11, IC3.4, IC5.11, IC5.4
- net TX0: no longer IC3.1, IC3.8, IC5.1, IC5.8
- net TX1: now also IC3.1, IC3.8, IC5.1, IC5.8
Routing:
- net +5V: track 0.00 -> 58.4 mm
- net TX1: track 0.00 -> 39.5 mm, vias 0 -> 4
- net H_LED: track 0.00 -> 31.2 mm, vias 0 -> 2
- net TX0: track 0.00 -> 29.6 mm, vias 0 -> 4
- net H_SET: track 0.00 -> 27.3 mm, vias 0 -> 4
- net G_SET: track 0.00 -> 25.7 mm, vias 0 -> 4
- net C_SET: track 0.00 -> 24.2 mm, vias 0 -> 2
- net G_LED: track 0.00 -> 23.7 mm, vias 0 -> 2
- net D_SET: track 0.00 -> 22.7 mm, vias 0 -> 2
- net RX1: track 0.00 -> 22.3 mm, vias 0 -> 2
- net N$14: track 0.00 -> 18.9 mm
- net N$3: track 0.00 -> 18.8 mm
- net N$32: track 0.00 -> 17.4 mm
- net N$33: track 0.00 -> 16.9 mm
- net N$37: track 0.00 -> 16.7 mm
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
Commit message: ditto
Signed-off-by: sosoru <siva6991@yahoo.co.jp>
Parts:
- moved Q1 2.93 mm to (40.5, 30.6)
- moved C8 2.19 mm to (41.8, 33.6)
- moved C7 2.19 mm to (38.3, 33.7)
- moved C1 1.29 mm to (40.2, 48.4), turned to 270 degrees
Routing:
- net +5V: track 58.4 -> 357.6 mm, vias 0 -> 9
- net !RESET: track 0.00 -> 83.3 mm, vias 0 -> 3
- net TX0: track 29.6 -> 95.6 mm, vias 4 -> 6
- net RX0: track 12.3 -> 73.8 mm, vias 0 -> 3
- net E_LED: track 0.00 -> 61.2 mm, vias 0 -> 4
- net F_LED: track 0.00 -> 51.8 mm, vias 0 -> 6
- net A_LED: track 0.00 -> 49.3 mm, vias 0 -> 4
- net D_LED: track 0.00 -> 47.5 mm, vias 0 -> 2
- net MOSI: track 0.00 -> 47.1 mm, vias 0 -> 1
- net MISO: track 0.00 -> 46.1 mm, vias 0 -> 2
- net VCC: track 0.00 -> 45.0 mm
- net !SS: track 0.00 -> 43.1 mm, vias 0 -> 2
- net SCK: track 0.00 -> 41.2 mm, vias 0 -> 1
- net E_SET: track 8.92 -> 46.4 mm, vias 2 -> 4
- net TMS: track 0.00 -> 34.9 mm, vias 0 -> 2
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