File: Schematics/EthControlling/MotorController.sch (EAGLE design)
At the start: 109 parts, among them IC1 TLP621-2, IC2 MEGA164P/324P/644P-AU, IC3 OPA4234P, IC4 TLP621-2, Q1 20.000M, T1 2SC1815, T2 2SC1815, T3 2SC1815, T4 2SC1815

Commit message: fix wiring of MotorController.sch and clear DRC errors
Signed-off-by: sosoru <siva6991@yahoo.co.jp>
Parts:
- added C28: 0.1u, rcl:C-EUC0603
- added R38, R39, R40, R41: 1Meg, resistor:R-EU_R0603
- C10, C16, C17, C9: value 0.47u -> 4.7u
- R10, R28, R29, R9: value 33k -> 3.3k
- R11, R12, R26, R27: value 0.01 -> 0.1
- R13, R14, R23, R24: value 100 -> 1k
Connections:
- net +5V: now also C28.2, JP1.4
- net GND: now also C28.1, R38.2, R39.2, R40.2, R41.2, U$1.P_GND, U$2.P_GND, U$3.P_GND, U$4.P_GND; no longer U$1.RSA, U$2.RSA, U$3.RSA, U$4.RSA
- net N$14: now also U$1.RSA; no longer U$1.P_GND
- net N$21: now also R38.1
- net N$30: now also R40.1
- net N$31: now also U$3.RSA; no longer U$3.P_GND
- net N$45: now also R39.1
- net N$46: now also U$2.RSA; no longer U$2.P_GND
- net N$60: now also R41.1
- net N$61: now also U$4.RSA; no longer U$4.P_GND
Other:
- moved on the sheet: C10, C3, C9, R10, R11, R12, R26, R27, R29, R9

Commit message: renumber MotorController.brd
Signed-off-by: sosoru <siva6991@yahoo.co.jp>
Parts:
- C10, C16, C6: value 4.7u -> 0.1u
- C11, C18, C24, C8: value 0.1u -> 4.7u
- C13: value 0.1u -> 100u; device rcl:C-EUC0603 -> rcl:CPOL-EUE2-5
- C14: value 100u -> 0.1u; device rcl:CPOL-EUE2-5 -> rcl:C-EUC0603
- C20: value 22p -> 0.1u
- C22: value 4.7u -> 22p
- C27: value (none) -> 0.1u; device rcl:CPOL-EUE2,5-6E -> rcl:C-EUC0603
- C28: value 0.1u -> (none); device rcl:C-EUC0603 -> rcl:CPOL-EUE2,5-6E
- R1: value 100k -> 3.3k
- R11: value 0.1 -> 3.3k; device resistor:R-EU_R1206 -> resistor:R-EU_R0603
- R13: value 1k -> 1Meg
- R14, R23: value 1k -> 3.3k
- R15: value 25k -> 0.1; device resistor:R-EU_R0603 -> resistor:R-EU_R1206
- R16: value 25k -> 3.3k
- R17: value 3.3k -> 1k
- R18, R20: value 3.3k -> 25k
- R19: value 10k -> 1k
- R2, R36, R37: value 10k -> 3.3k
- R22: value 25k -> 10k
- R24: value 1k -> 25k
- R25: value 25k -> 1k
- R26: value 0.1 -> 1k; device resistor:R-EU_R1206 -> resistor:R-EU_R0603
- R27: value 0.1 -> 25k; device resistor:R-EU_R1206 -> resistor:R-EU_R0603
- R28: value 3.3k -> 1Meg
- R29: value 3.3k -> 0.1; device resistor:R-EU_R0603 -> resistor:R-EU_R1206
- R3: value 500 -> 1Meg
- R34: value 100k -> 1Meg
- R35: value 100k -> 0.1; device resistor:R-EU_R0603 -> resistor:R-EU_R1206
- R38, R40: value 1Meg -> 100k
- R39, R41: value 1Meg -> 10k
- R4: value 10k -> 100k
- R5: value 500 -> 10k
- R6: value 100k -> 500
- R7: value 3.3k -> 500
- R8: value 3.3k -> 10k
- R9: value 3.3k -> 100k
Connections:
- removed net N$14 (its old number): R11.1, R9.1, U$1.RSA
- new net N$46: R15.1, R2.1, U$1.RSA
- net !RESET: now also R22.2; no longer R19.2
- net +5V: now also C10.2, C13.+, C14.2, C16.2, R22.1; no longer C11.2, C13.2, C14.+, C28.2, R19.1
- net A_OUT1: now also R16.2, U$2.OUT1; no longer R17.2, U$1.OUT1
- net A_OUT2: now also U$2.OUT2; no longer U$1.OUT2
- net A_OUT3: now also R21.2; no longer R20.2
- net A_OUT5: now also R14.2, U$1.OUT1; no longer R18.2, U$2.OUT1
- net A_OUT6: now also U$1.OUT2; no longer U$2.OUT2
- net A_OUT7: now also R23.2; no longer R21.2
- net CTRL_A_1: now also U$2.IN1; no longer U$1.IN1
- net CTRL_A_2: now also U$2.IN2; no longer U$1.IN2
- net CTRL_A_3: now also R6.1, U$2.SB; no longer R3.1, U$1.SB
- net CTRL_A_ALERT: now also C8.1, R11.2; no longer C5.1, R7.2
- net CTRL_A_PWM: now also U$2.OSC/PWM; no longer U$1.OSC/PWM
- net CTRL_B_1: now also U$1.IN1; no longer U$2.IN1
- net CTRL_B_2: now also U$1.IN2; no longer U$2.IN2
- net CTRL_B_3: now also R7.1, U$1.SB; no longer R5.1, U$2.SB
- net CTRL_B_ALERT: now also C5.1, R1.2; no longer C6.1, R8.2
- net CTRL_B_PWM: now also U$1.OSC/PWM; no longer U$2.OSC/PWM
- net CTRL_C_ALERT: now also C18.1, R31.2; no longer C22.1, R30.2
- net CTRL_D_ALERT: now also C24.1, R37.2; no longer C23.1, R31.2
- net FEEDBACK_A: now also R20.2; no longer R16.2
- net FEEDBACK_B: now also R18.2; no longer R15.2
- net FEEDBACK_C: now also R27.2; no longer R25.2
- net FEEDBACK_D: now also R24.2; no longer R22.2
- net GND: now also C10.1, C11.2, C13.-, C14.1, C16.1, C18.2, C19.2, C22.1, C25.1, C27.2, C28.-, C3.1, C6.1, C7.2, C8.2, R15.2, R17.2, R19.2, R25.2, R28.2, R29.2, R3.2, R4.2, R9.2; no longer C10.2, C11.1, C13.1, C14.-, C16.2, C18.1, C19.1, C22.2, C25.2, C27.-, C28.1, C3.2, C6.2, C7.1, C8.1, R1.2, R11.2, R14.2, R23.2, R24.2, R27.2, R39.2, R41.2, R6.2
- net N$10: now also C2.+, C6.2, U$2.VCC; no longer C1.+, C7.2, U$1.VCC
- net N$11: now also R19.1, R20.1; no longer R14.1, R16.1
- net N$12: now also R31.1; no longer R30.1
- net N$18: now also C20.2, C26.+; no longer C18.2, C27.+
- net N$19: now also R21.1; no longer R20.1
- net N$20: now also R7.2; no longer R5.2
- net N$21: now also C11.1, R10.2, R13.1; no longer C9.1, R38.1, R9.2
- net N$26: now also R38.1, R39.1; no longer R35.1, R36.1
- net N$28: now also R39.2; no longer R36.2
- net N$29: now also R26.1, R27.1; no longer R24.1, R25.1
- net N$3: now also C22.2; no longer C20.2
- net N$30: now also C17.1, R28.1, R30.2; no longer C16.1, R28.2, R40.1
- net N$31: now also R29.1, R30.1; no longer R26.1, R28.1
- net N$32: now also U$1.VREG; no longer U$2.VREG
- net N$33: now also R1.1, U$1.ALERT; no longer R8.1, U$2.ALERT
- net N$34: now also C1.+, C3.2, U$1.VCC; no longer C2.+, C8.2, U$2.VCC
- net N$35: now also R14.1; no longer R18.1
- net N$4: now also R11.1, U$2.ALERT; no longer R7.1, U$1.ALERT
- net N$41: now also R5.1; no longer R1.1
- net N$42: now also D1.C; no longer D2.C
- net N$43: now also R5.2; no longer R4.2
- net N$44: now also R17.1, R18.1; no longer R13.1, R15.1
- net N$45: now also C9.1, R2.2, R3.1; no longer C10.1, R10.2, R39.1
- net N$47: now also C27.1; no longer C25.1
- net N$48: now also R37.1; no longer R31.1
- net N$49: now also C25.2, C28.+; no longer C19.2, C26.+
- net N$5: now also C7.1, U$2.VREG; no longer C3.1, U$1.VREG
- net N$50: now also R23.1; no longer R21.1
- net N$56: now also R40.1, R41.1; no longer R34.1, R37.1
- net N$58: now also R41.2; no longer R37.2
- net N$59: now also R24.1, R25.1; no longer R22.1, R23.1
- net N$6: now also R6.2; no longer R3.2
- net N$60: now also C23.1, R34.1, R36.2; no longer C17.1, R29.2, R41.1
- net N$61: now also R35.1, R36.1; no longer R27.1, R29.1
- net N$7: now also R8.1, R9.1; no longer R2.1, R6.1
- net N$8: now also R16.1; no longer R17.1
- net N$84: now also D2.C; no longer D1.C
- net N$86: now also R8.2; no longer R2.2
- net N$9: now also C19.1; no longer C24.1
Other:
- moved on the sheet: C1, C10, C11, C15, C16, C17, C18, C19, C2, C20, C22, C23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

Commit message: ditto
Signed-off-by: sosoru <siva6991@yahoo.co.jp>
Parts:
- R32, R33, R6, R7: value 500 -> 1k
Changed lines of the file:
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@@
 <part name="LED3" library="led" deviceset="LED" device="3MM" value="G"/>
 <part name="R16" library="resistor" deviceset="R-EU_" device="R0603" value="3.3k"/>
-<part name="R6" library="resistor" deviceset="R-EU_" device="R0603" value="500"/>
+<part name="R6" library="resistor" deviceset="R-EU_" device="R0603" value="1k"/>
 <part name="GND8" library="supply1" deviceset="GND" device=""/>
 <part name="P+7" library="supply1" deviceset="+12V" device=""/>
@@
 <part name="LED5" library="led" deviceset="LED" device="3MM" value="G"/>
 <part name="R21" library="resistor" deviceset="R-EU_" device="R0603" value="3.3k"/>
-<part name="R32" library="resistor" deviceset="R-EU_" device="R0603" value="500"/>
+<part name="R32" library="resistor" deviceset="R-EU_" device="R0603" value="1k"/>
 <part name="GND16" library="supply1" deviceset="GND" device=""/>
 <part name="P+12" library="supply1" deviceset="+12V" device=""/>
@@
 <part name="LED1" library="led" deviceset="LED" device="3MM" value="G"/>
 <part name="R14" library="resistor" deviceset="R-EU_" device="R0603" value="3.3k"/>
-<part name="R7" library="resistor" deviceset="R-EU_" device="R0603" value="500"/>
+<part name="R7" library="resistor" deviceset="R-EU_" device="R0603" value="1k"/>
 <part name="GND26" library="supply1" deviceset="GND" device=""/>
 <part name="P+17" library="supply1" deviceset="+12V" device=""/>
@@
 <part name="LED7" library="led" deviceset="LED" device="3MM" value="G"/>
 <part name="R23" library="resistor" deviceset="R-EU_" device="R0603" value="3.3k"/>
-<part name="R33" library="resistor" deviceset="R-EU_" device="R0603" value="500"/>
+<part name="R33" library="resistor" deviceset="R-EU_" device="R0603" value="1k"/>
 <part name="GND35" library="supply1" deviceset="GND" device=""/>
 <part name="P+22" library="supply1" deviceset="+12V" device=""/>

Commit message: fix resistor value of MotorController
Signed-off-by: sosoru <siva6991@yahoo.co.jp>
Parts:
- R18, R20, R24, R27: value 25k -> 33k
Changed lines of the file:
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@@
 <part name="R12" library="resistor" deviceset="R-EU_" device="R1206" value="0.1"/>
 <part name="R19" library="resistor" deviceset="R-EU_" device="R0603" value="1k"/>
-<part name="R20" library="resistor" deviceset="R-EU_" device="R0603" value="25k"/>
+<part name="R20" library="resistor" deviceset="R-EU_" device="R0603" value="33k"/>
 <part name="GND10" library="supply1" deviceset="GND" device=""/>
 <part name="GND11" library="supply1" deviceset="GND" device=""/>
@@
 <part name="R29" library="resistor" deviceset="R-EU_" device="R1206" value="0.1"/>
 <part name="R26" library="resistor" deviceset="R-EU_" device="R0603" value="1k"/>
-<part name="R27" library="resistor" deviceset="R-EU_" device="R0603" value="25k"/>
+<part name="R27" library="resistor" deviceset="R-EU_" device="R0603" value="33k"/>
 <part name="GND19" library="supply1" deviceset="GND" device=""/>
 <part name="R30" library="resistor" deviceset="R-EU_" device="R0603" value="3.3k"/>
@@
 <part name="R15" library="resistor" deviceset="R-EU_" device="R1206" value="0.1"/>
 <part name="R17" library="resistor" deviceset="R-EU_" device="R0603" value="1k"/>
-<part name="R18" library="resistor" deviceset="R-EU_" device="R0603" value="25k"/>
+<part name="R18" library="resistor" deviceset="R-EU_" device="R0603" value="33k"/>
 <part name="GND28" library="supply1" deviceset="GND" device=""/>
 <part name="R2" library="resistor" deviceset="R-EU_" device="R0603" value="3.3k"/>
@@
 <part name="R35" library="resistor" deviceset="R-EU_" device="R1206" value="0.1"/>
 <part name="R25" library="resistor" deviceset="R-EU_" device="R0603" value="1k"/>
-<part name="R24" library="resistor" deviceset="R-EU_" device="R0603" value="25k"/>
+<part name="R24" library="resistor" deviceset="R-EU_" device="R0603" value="33k"/>
 <part name="GND37" library="supply1" deviceset="GND" device=""/>
 <part name="R36" library="resistor" deviceset="R-EU_" device="R0603" value="3.3k"/>
