File: Schematics/EthControlling/AtxPowerDispatcher3.sch (EAGLE design)
At the start: 44 parts, among them IC2 788TV, IC3 SI-8050, J2 ATX24RH, X1 DCJACK--H3, X2 DCJACK--H3, X3 DCJACK--H3

Commit message: Submit AtxPowerDispatcher3
Parts:
- removed D6, D7, D8, D9: 1N4148DO35-7, diode:1N4148DO35-7
- removed IC3: SI-8050, myparts:SI-8050
- added D1, D2, D3, D4: 1N5817-B, diode:1N5817-B
- added IC1: 788TV, myparts:788TV
- C3: value 100u -> 0.1u; device rcl:CPOL-EUE2,5-6E -> rcl:C-EUC0603
- C4: value 0.1u -> 100u; device rcl:C-EUC0603 -> rcl:CPOL-EUE2,5-6E
- C5: value 10u -> 0.1u; device rcl:C-EUC1206 -> rcl:C-EUC0603
- C6, C7: device rcl:CPOL-EUE2,5-6E -> rcl:CPOL-EUE5-10.5
- C9: value 0.1u -> 10u; device rcl:C-EUC0603 -> rcl:C-EUC1206
- D5: value 1N4148DO35-7 -> 1N4728; device diode:1N4148DO35-7 -> diode:1N4728
- IC2: value 788TV -> SI-8050; device myparts:788TV -> myparts:SI-8050
- R1: value 1k -> 30 5W; device rcl:R-EU_R0603 -> resistor:R-EU_0922/22
- R2, R3: value 1k -> 5 5W; device rcl:R-EU_R0603 -> resistor:R-EU_0922/22
- R4, R5: value 5 5W -> 1k; device resistor:R-EU_0922/22 -> rcl:R-EU_R0603
- R6: value 30 5W -> 1k; device resistor:R-EU_0922/22 -> rcl:R-EU_R0603
- X1, X2, X3: value DCJACK--H3 -> DCJACK; device kamiki-dcjack:DCJACK--H3 -> kamiki-dcjack:DCJACK
- renumbered J2 to J1, L2 to L1
Connections:
- net +12V: now also C5.1, D1.C, D3.C, D4.C, IC1.VI, IC2.VIN, R5.2; no longer C8.1, D5.C, D8.C, D9.C, IC2.VI, IC3.VIN, R1.2
- net +5V: now also C8.1, D3.A, IC2.VOS, R6.2; no longer C9.1, D8.A, IC3.VOS, R2.2
- net 3.3V: now also C3.1, C4.+, D1.A, IC1.VO, R7.2; no longer C3.+, C4.1, D5.A, IC2.VO, R3.2
- net GND: now also C3.2, C4.-, D5.A, IC1.GND, R2.1, R3.1; no longer C3.-, C4.2, D6.A, IC3.GND, R4.1, R5.1
- net N$1: now also R5.1; no longer R1.1
- net N$10: now also D2.A, R1.1; no longer D7.A, R6.1
- net N$11: now also D2.C, R1.2; no longer D7.C, R6.2
- net N$17: now also C9.1, IC2.S.S; no longer C5.1, IC3.S.S
- net N$2: now also R4.2; no longer R7.2
- net N$3: now also R2.2, R3.2; no longer R4.2, R5.2
- net N$4: now also R6.1; no longer R2.1
- net N$5: now also R7.1; no longer R3.1
- net N$6: now also R4.1; no longer R7.1
- net N$8: now also D4.A; no longer D9.A
- net N$9: now also D5.C, IC2.SWOUT; no longer D6.C, IC3.SWOUT
Other:
- moved on the sheet: C5, C8, C9, R1, R2, R3, R4, R5, R6, R7
