File: Schematics/submitted/2014_1009_AtcPowerDispatcher_forFusionPcb/AtxPowerDispatcher3.brd (EAGLE design)
At the start: 100 x 50 mm, 44 parts, among them IC2 788TV, IC3 SI-8050, J2 ATX24RH, X1 DCJACK--H3, X2 DCJACK--H3, X3 DCJACK--H3

Commit message: Submit AtxPowerDispatcher3
Parts:
- removed D6, D7, D8, D9: 1N4148DO35-7, diode:DO35-7
- removed IC3: SI-8050, myparts:TO220-5
- added D1, D2, D3, D4: 1N5817-B, diode:DO41-7.6
- added IC1: 788TV, myparts:TO220V
- C3: value 100u -> 0.1u; device rcl:E2,5-6E -> rcl:C0603
- C4: value 0.1u -> 100u; device rcl:C0603 -> rcl:E2,5-6E
- C5: value 10u -> 0.1u; device rcl:C1206 -> rcl:C0603
- C6, C7: device rcl:E2,5-6E -> rcl:E5-10,5
- C9: value 0.1u -> 10u; device rcl:C0603 -> rcl:C1206
- D5: value 1N4148DO35-7 -> 1N4728; device diode:DO35-7 -> diode:DO41Z10
- IC2: value 788TV -> SI-8050; device myparts:TO220V -> myparts:TO220-5
- R1: value 1k -> 30 5W; device rcl:R0603 -> resistor:0922/22
- R2, R3: value 1k -> 5 5W; device rcl:R0603 -> resistor:0922/22
- R4, R5: value 5 5W -> 1k; device resistor:0922/22 -> rcl:R0603
- R6: value 30 5W -> 1k; device resistor:0922/22 -> rcl:R0603
- X1, X2, X3: value DCJACK--H3 -> DCJACK; device kamiki-dcjack:2DC-0005D100--H3 -> kamiki-dcjack:2DC-0005D100
- moved R2 57.3 mm to (37.6, 22.9), flipped to the bottom, turned to 270 degrees
- moved R3 41.0 mm to (55.9, 25.4), flipped to the bottom, turned to 270 degrees
- moved R5 39.4 mm to (94.0, 15.2), flipped to the top, turned to 0 degrees
- moved R4 33.1 mm to (69.8, 15.2), flipped to the top, turned to 0 degrees
- moved IC2 26.9 mm to (29.2, 44.5)
- moved D5 26.4 mm to (39.4, 29.2)
- moved R7 24.7 mm to (94.0, 10.2)
- moved R6 23.3 mm to (94.0, 12.7), flipped to the top, turned to 0 degrees
- moved R1 21.6 mm to (77.5, 29.2), flipped to the bottom, turned to 270 degrees
- moved C9 15.5 mm to (43.2, 26.7), turned to 270 degrees
- moved C4 14.8 mm to (40.6, 17.8), turned to 0 degrees
- moved C5 14.1 mm to (24.9, 33.3), turned to 0 degrees
- moved C1 12.3 mm to (21.6, 13.2), turned to 270 degrees
- moved JP3.3V 11.4 mm to (31.8, 19.1), turned to 90 degrees
- moved C3 9.18 mm to (32.0, 8.89), turned to 180 degrees
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- renumbered J2 to J1, L2 to L1
Connections:
- net +12V: now also C5.1, D1.C, D3.C, D4.C, IC1.1, R5.2; no longer C8.1, D5.C, D8.C, D9.C, IC3.1, R1.2
- net +5V: now also C8.1, D3.A, IC2.4, R6.2; no longer C9.1, D8.A, IC3.4, R2.2
- net 3.3V: now also C3.1, C4.+, D1.A, IC1.3, R7.2; no longer C3.+, C4.1, D5.A, IC2.3, R3.2
- net GND: now also C3.2, C4.-, D5.A, IC1.2, IC2.3, R2.1, R3.1; no longer C3.-, C4.2, D6.A, IC2.2, IC3.3, R4.1, R5.1
- net N$1: now also R5.1; no longer R1.1
- net N$10: now also D2.A, R1.1; no longer D7.A, R6.1
- net N$11: now also D2.C, R1.2; no longer D7.C, R6.2
- net N$17: now also C9.1, IC2.5; no longer C5.1, IC3.5
- net N$2: now also R4.2; no longer R7.2
- net N$3: now also R2.2, R3.2; no longer R4.2, R5.2
- net N$4: now also R6.1; no longer R2.1
- net N$5: now also R7.1; no longer R3.1
- net N$6: now also R4.1; no longer R7.1
- net N$8: now also D4.A; no longer D9.A
- net N$9: now also D5.C, IC2.2; no longer D6.C, IC3.2
Routing:
- net N$11: track 166.7 -> 177.8 mm, vias 15 -> 12
- net N$9: track 27.3 -> 35.6 mm
- net 3.3V: track 167.9 -> 175.5 mm
- net +12V: track 170.9 -> 176.3 mm
- net +5V: track 174.1 -> 178.0 mm
- net N$17: track 12.0 -> 15.6 mm
